Commit message: Added robot_state_publisher to launch file using the URDF file instead of the TF in the sensor node file which are commented out for now

File: urdfs/roborama25.urdf (robot description, URDF)
Before this commit: robot roborama25, 13 links, 12 joints
Links:
- removed link base_rangef
- removed link base_rangerc
- removed link base_rangerl
- removed link base_rangerr
- removed link base_scan
- removed link base_scanl
- removed link base_scanr
- added link lidar_link; visual cylinder length=0.020 radius=0.025
- added link tofL4_link; visual box size=0.005 0.025 0.025
- added link tofL5L_link; visual cylinder length=0.030 radius=0.020
- added link tofL5R_link; visual cylinder length=0.030 radius=0.020
- added link tofRC_link; visual cylinder length=0.005 radius=0.015
- added link tofRL_link; visual cylinder length=0.005 radius=0.015
- added link tofRR_link; visual cylinder length=0.005 radius=0.015
Joints:
- removed joint range_jointf
- removed joint range_jointrc
- removed joint range_jointrl
- removed joint range_jointrr
- removed joint scan_joint
- removed joint scan_jointl
- removed joint scan_jointr
- added joint lidar_joint: type fixed, parent base_link, child lidar_link, origin xyz=0 0 0.115 rpy=0 0 3.1416
- added joint tofL4_joint: type fixed, parent base_link, child tofL4_link, origin xyz=0.100 0 0.030 rpy=0 0 0
- added joint tofL5L_joint: type fixed, parent base_link, child tofL5L_link, origin xyz=0.140 0.060 0.030 rpy=0 0 0.41
- added joint tofL5R_joint: type fixed, parent base_link, child tofL5R_link, origin xyz=0.140 -0.060 0.030 rpy=0 0 -0.41
- added joint tofRC_joint: type fixed, parent base_link, child tofRC_link, origin xyz=-0.040 0 0.085 rpy=0 0 3.1416
- added joint tofRL_joint: type fixed, parent base_link, child tofRL_link, origin xyz=-0.040 0 0.085 rpy=0 0 2.3
- added joint tofRR_joint: type fixed, parent base_link, child tofRR_link, origin xyz=-0.040 0 0.085 rpy=0 0 -2.3

Commit message: wheel controller node now working with robot state TF

File: urdfs/roborama25.urdf (robot description, URDF)
Before this commit: robot roborama25, 13 links, 12 joints
Links:
- added link map
- added link odom
Joints:
- removed joint base_joint
- added joint base_footprint_joint: type fixed, parent odom, child base_footprint, origin xyz=0 0 0 rpy=0 0 0
- added joint base_link_joint: type fixed, parent base_footprint, child base_link, origin xyz=0 0 0.042 rpy=0 0 0
- added joint odom_joint: type fixed, parent map, child odom, origin xyz=0 0 0 rpy=0 0 0
